Commit message: adding lidar but not done

File: src/assem1_v4/urdf/assem1_v4.urdf (robot description, URDF)
Before this commit: robot assem1_v3, 5 links, 4 joints
Links:
- added link Ball_back_link, mass 0.00525183168276762; collision mesh filename=package://assem1_v4/meshes/Ball_back_link.STL; visual mesh filename=package://assem1_v4/meshes/Ball_back_link.STL
- added link Ball_front_link, mass 0.00525183168276763; collision mesh filename=package://assem1_v4/meshes/Ball_front_link.STL; visual mesh filename=package://assem1_v4/meshes/Ball_front_link.STL
- link L_wheel_link: mass 0.0419551495558707 -> 0.0419551495558706; geometry collision mesh filename=package://assem1_v4/meshes/L_wheel_link.STL; visual mesh filename=package://assem1_v4/meshes/L_wheel_link.STL
- link Lidar_link: mass 0.031240912686575 -> 0.0312409126861326; geometry collision mesh filename=package://assem1_v4/meshes/Lidar_link.STL; visual mesh filename=package://assem1_v4/meshes/Lidar_link.STL
- link R_wheel_link: mass 0.0419551495558989 -> 0.0419551495559627; geometry collision mesh filename=package://assem1_v4/meshes/R_wheel_link.STL; visual mesh filename=package://assem1_v4/meshes/R_wheel_link.STL
- link base_link: geometry collision mesh filename=package://assem1_v4/meshes/base_link.STL; visual mesh filename=package://assem1_v4/meshes/base_link.STL
- link imu_link: geometry collision mesh filename=package://assem1_v4/meshes/imu_link.STL; visual mesh filename=package://assem1_v4/meshes/imu_link.STL
Joints:
- added joint Ballback_joint: type fixed, parent base_link, child Ball_back_link, origin xyz=-0.0754043917543321 -0.000183494055149433 0.00159999999999952 rpy=0 0 0, axis 0 0 0
- added joint Ballfront_joint: type fixed, parent base_link, child Ball_front_link, origin xyz=0.074595608245668 -0.000183494055149488 0.00159999999999952 rpy=0 0 0, axis 0 0 0
